File: Neat Snicket-Gaaris.brd (EAGLE design)
At the start: 264.8 x 214.6 mm, 17 parts, among them U3 ARDUINO-UNO-R3-SHIELD, U4 TMP36GT9Z_TO92, U5 LCD-16X2JHD-162A

Commit message: Controlled temperature with light bulb source
Parts:
- removed S1, S2, S3, S4: SWITCH_MOMENTARY, Tinkercad:SWITCH-MOMENTARY-PTH-6.5MM
- removed U4: TMP36GT9Z_TO92, Tinkercad:TO92
- added L1: LIGHTBULB, Tinkercad:1X02
- added P1: BATTERYGENERIC, Tinkercad:BATTERY-GENERIC
- added S6, S7, S8, S9: SWITCH_MOMENTARY, Tinkercad:SWITCH-MOMENTARY-PTH-6.5MM
- added T1: NMOSFET, Tinkercad:TO220BV
- added UTEMP_SENSOR: TMP36GT9Z_TO92, Tinkercad:TO92
- moved R7 197.4 mm to (58.7, 26.9)
- moved R8 197.4 mm to (58.7, 9.08)
- moved R1 146.6 mm to (88.7, 26.8)
- moved R2 146.6 mm to (88.7, 8.97)
- moved R3 132.5 mm to (73.3, 27.1)
- moved R4 132.5 mm to (73.3, 9.35)
- moved R5 128.0 mm to (99.0, 27.0)
- moved R6 128.0 mm to (99.0, 9.20)
- moved RRESISTOR 8.50 mm to (146.5, 174.5)
- moved U3 8.50 mm to (47.9, 158.8)
- moved U5 8.50 mm to (127.6, 106.1)
- moved BAT1 8.50 mm to (230.1, 214.9)
Connections:
- removed net S1_2: R1.1, R2.2, S1.1, S1.2
- removed net S2_2: R3.1, R4.2, S2.1, S2.2
- removed net S3_2: R5.1, R6.2, S3.1, S3.2
- removed net S4_2: R7.1, R8.2, S4.1, S4.2
- new net L1_1: L1.1, T1.D
- new net P1+: L1.2, P1.+
- new net S6_2: R7.1, R8.2, S6.1, S6.2
- new net S7_2: R3.1, R4.2, S7.1, S7.2
- new net S8_2: R1.1, R2.2, S8.1, S8.2
- new net S9_2: R5.1, R6.2, S9.1, S9.2
- new net U3_D10: T1.G, U3.D10
- net BAT1+: now also UTEMP_SENSOR.3; no longer U4.3
- net BAT1-: now also P1.-, T1.S, UTEMP_SENSOR.1; no longer U4.1
- net U3_5V: now also S6.3, S7.3, S8.3, S9.3; no longer S1.3, S2.3, S3.3, S4.3
- net U3_A0: now also UTEMP_SENSOR.2; no longer U4.2
Other:
- board size 264.8 x 214.6 mm -> 248.3 x 230.2 mm
